File: esp32-h2-thtkit/esp32-h2-thtkit.kicad_pcb (KiCad board)
At the start: 4 copper layers, 0 parts

Commit message: Basic components layout
Parts:
- added AE1: Antenna_Chip, PCM_SKC_Antennas_SMD:Antenna_PCB_Espressif_2.4GHz_Left, F.Cu at (136.6, 91.6)
- added C10: 100n 6.3V X7R, Capacitor_SMD:C_0402_1005Metric, F.Cu at (141.0, 99.7)
- added C11: 8p 6.3V C0G, Capacitor_SMD:C_0201_0603Metric, F.Cu at (141.3, 103.7)
- added C12: 1m 6.3V X7R, Capacitor_SMD:C_0402_1005Metric, F.Cu at (132.6, 95.3)
- added C13: 470p 6.3V X7R, Capacitor_SMD:C_0201_0603Metric, F.Cu at (131.9, 100.7)
- added C15: 2.2m 6.3V TANT, Capacitor_Tantalum_SMD:CP_EIA-2012-12_Kemet-R, F.Cu at (133.2, 101.7)
- added C3: 100n 6.3V X7R, Capacitor_SMD:C_0402_1005Metric, F.Cu at (140.4, 96.3)
- added C4: 5.6p C0G, Capacitor_SMD:C_0201_0603Metric, F.Cu at (141.3, 96.3)
- added C5: 100n 6.3V X7R, Capacitor_SMD:C_0402_1005Metric, F.Cu at (137.2, 95.3)
- added C6: 2.2p C0G, Capacitor_SMD:C_0201_0603Metric, F.Cu at (141.7, 95.2)
- added C7: 100n 6.3V X7R, Capacitor_SMD:C_0402_1005Metric, F.Cu at (135.1, 100.7)
- added C8: 8p 6.3V C0G, Capacitor_SMD:C_0201_0603Metric, F.Cu at (143.2, 102.4)
- added C9: 100n 6.3V X7R, Capacitor_SMD:C_0402_1005Metric, F.Cu at (139.3, 102.0)
- added J1: PIN_GROUP_1, PCM_SKC_Connector_PinHeader_2.54mm:PinHeader_1x06_P2.54mm_Vertical_NoSilk, B.Cu at (130.2, 96.7)
- added J2: PIN_GROUP_2, PCM_SKC_Connector_PinHeader_2.54mm:PinHeader_1x06_P2.54mm_Vertical_NoSilk, B.Cu at (145.4, 96.7)
- added J3: UART, Connector_PinHeader_2.54mm:PinHeader_1x04_P2.54mm_Vertical, F.Cu at (134.0, 106.8)
- added J6: PIN_GROUP_3, PCM_SKC_Connector_PinHeader_2.54mm:PinHeader_1x04_P2.54mm_Vertical_NoSilk, B.Cu at (134.0, 109.4)
- added L1: 3.9 nH, Inductor_SMD:L_0402_1005Metric, F.Cu at (141.8, 97.6)
- added R1: 10k, Resistor_SMD:R_0402_1005Metric, F.Cu at (132.9, 104.1)
- added R2: 10k, Resistor_SMD:R_0402_1005Metric, F.Cu at (138.8, 104.1)
- added TP1: TestPoint_2Pole, TestPoint:TestPoint_Pad_D1.0mm, F.Cu at (134.8, 104.1)
- added TP2: TestPoint_2Pole, TestPoint:TestPoint_Pad_D1.0mm, F.Cu at (136.9, 104.1)
- added U2: ESP32-H2, PCM_SKC_MCU_Espressif:TQFN_32_1EP_4x4mm_P0.4mm_EP2.4x2.4mm_Compact, F.Cu at (137.8, 98.8)
- added U3: MIC5219-3.3YM5, Package_TO_SOT_SMD:SOT-23-5, F.Cu at (133.0, 97.9)
- added Y1: 32MHz ±10ppm CL8pF, Crystal:Crystal_SMD_2016-4Pin_2.0x1.6mm, F.Cu at (141.3, 102.0)
Routing:
- net /RF: track 0.00 -> 3.12 mm
- net Net-(AE1-FEED): track 0.00 -> 1.56 mm
- net +3.3V: track 0.00 -> 1.54 mm
Other:
- board outline added: 17.9 x 21.9 mm
